File: circuit/7G_controller.brd (EAGLE design)
At the start: 63 x 70.5 mm, 23 parts, among them Q1 32768Hz, T1 TPS1101D

Commit message: finished adding the CR2032 battery holder
Parts:
- removed U$1: (no value), adafruit:CR2032-SMD
- added BATT_CR2032: (no value), KileParts:CR2032-SMD
Connections:
- net GND: now also BATT_CR2032.-; no longer U$1.-
- net N$4: now also BATT_CR2032.+$1, BATT_CR2032.+$2; no longer U$1.+$1, U$1.+$2
Routing:
- net N$4: track 25.0 -> 113.3 mm
- net GND: track 223.7 -> 251.8 mm
Changed lines of the file:
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@@
 <setting verticaltext="up"/>
 </settings>
-<grid distance="0.00625" unitdist="inch" unit="inch" style="lines" multiple="1" display="yes" altdistance="0.025" altunitdist="inch" altunit="inch"/>
+<grid distance="0.0125" unitdist="inch" unit="inch" style="lines" multiple="1" display="yes" altdistance="0.025" altunitdist="inch" altunit="inch"/>
 <layers>
 <layer number="1" name="Top" color="4" fill="1" visible="yes" active="yes"/>
@@
 <layer number="19" name="Unrouted" color="6" fill="1" visible="yes" active="yes"/>
 <layer number="20" name="Dimension" color="15" fill="1" visible="yes" active="yes"/>
-<layer number="21" name="tPlace" color="7" fill="1" visible="yes" active="yes"/>
+<layer number="21" name="tPlace" color="7" fill="1" visible="no" active="yes"/>
 <layer number="22" name="bPlace" color="7" fill="1" visible="yes" active="yes"/>
-<layer number="23" name="tOrigins" color="15" fill="1" visible="yes" active="yes"/>
+<layer number="23" name="tOrigins" color="15" fill="1" visible="no" active="yes"/>
 <layer number="24" name="bOrigins" color="15" fill="1" visible="yes" active="yes"/>
-<layer number="25" name="tNames" color="7" fill="1" visible="yes" active="yes"/>
+<layer number="25" name="tNames" color="7" fill="1" visible="no" active="yes"/>
 <layer number="26" name="bNames" color="7" fill="1" visible="yes" active="yes"/>
 <layer number="27" name="tValues" color="7" fill="1" visible="no" active="yes"/>
@@
 <layer number="46" name="Milling" color="3" fill="1" visible="no" active="yes"/>
 <layer number="47" name="Measures" color="7" fill="1" visible="no" active="yes"/>
-<layer number="48" name="Document" color="7" fill="1" visible="yes" active="yes"/>
+<layer number="48" name="Document" color="7" fill="1" visible="no" active="yes"/>
 <layer number="49" name="Reference" color="7" fill="1" visible="no" active="yes"/>
 <layer number="50" name="dxf" color="7" fill="1" visible="no" active="no"/>
-<layer number="51" name="tDocu" color="7" fill="1" visible="yes" active="yes"/>
+<layer number="51" name="tDocu" color="7" fill="1" visible="no" active="yes"/>
 <layer number="52" name="bDocu" color="7" fill="1" visible="yes" active="yes"/>
 <layer number="53" name="tGND_GNDA" color="7" fill="9" visible="no" active="no"/>
@@
 <attribute name="OC_FARNELL" value="unknown" x="48.26" y="18.51" size="1.778" layer="27" display="off"/>
 </element>
-<element name="U$1" library="adafruit" package="CR2032-SMD" value="" x="10" y="42" rot="MR270"/>
+<element name="BATT_CR2032" library="KileParts" package="CR2032-SMD" value="" x="10" y="42" rot="MR270"/>
 </elements>
 <signals>
@@
 <wire x1="52.07" y1="21.235" x2="52.07" y2="18.51" width="0.254" layer="1"/>
 <wire x1="31.4325" y1="35.08375" x2="35.40125" y2="35.08375" width="0.254" layer="1"/>
-<contactref element="U$1" pad="-"/>
-<wire x1="10" y1="42" x2="10.4775" y2="6.985" width="0" layer="19" extent="1-1"/>
+<contactref element="BATT_CR2032" pad="-"/>
+<wire x1="10.7" y1="61.58" x2="14.605" y2="61.58" width="0.4064" layer="16"/>
+<wire x1="14.605" y1="61.58" x2="14.605" y2="42" width="0.4064" layer="16"/>
+<wire x1="14.605" y1="42" x2="10" y2="42" width="0.4064" layer="16"/>
 </signal>
 <signal name="MOSI">
@@
 <wire x1="57.54" y1="17.425" x2="59.3725" y2="17.425" width="0.254" layer="1"/>
 <wire x1="59.3725" y1="17.425" x2="59.3725" y2="32.325" width="0.254" layer="1"/>
-<contactref element="U$1" pad="+$1"/>
-<contactref element="U$1" pad="+$2"/>
-<wire x1="10" y1="29.3" x2="57.5945" y2="13.0175" width="0" layer="19" extent="1-1"/>
-<wire x1="10" y1="54.7" x2="10" y2="29.3" width="0" layer="19" extent="1-1"/>
+<contactref element="BATT_CR2032" pad="+$1"/>
+<contactref element="BATT_CR2032" pad="+$2"/>
+<wire x1="10" y1="29.3" x2="10" y2="13.6525" width="0.4064" layer="16"/>
+<wire x1="10" y1="13.6525" x2="7.9375" y2="13.6525" width="0.4064" layer="16"/>
+<wire x1="7.9375" y1="13.6525" x2="7.9375" y2="5.08" width="0.4064" layer="16"/>
+<wire x1="7.9375" y1="5.08" x2="54.61" y2="5.08" width="0.4064" layer="16"/>
+<wire x1="54.61" y1="5.08" x2="54.61" y2="17.4625" width="0.4064" layer="16"/>
+<wire x1="54.61" y1="17.4625" x2="57.54" y2="17.4625" width="0.4064" layer="16"/>
+<wire x1="57.54" y1="17.4625" x2="57.54" y2="17.425" width="0.4064" layer="16"/>
+<wire x1="10" y1="29.3" x2="10" y2="54.7" width="0" layer="19" extent="16-16"/>
 </signal>
 <signal name="N$6">
